Commit message: Addition of files for the Andreas Arm control

File: urdf/andreas_arm_description.xacro (robot description, xacro)
@@ -47,4 +47,5 @@
     <xacro:property name="zetaJointRadius"     value=".027" />
     <xacro:property name="zetaJointZ"          value=".005" />
+    <xacro:property name="endEffectorZ"        value=".010" />
     <material name="brown">
         <color rgba="${255/255} ${185/255} ${  0/255} ${255/255}" />
@@ -185,4 +186,9 @@
         <xacro:defaultInertial mass="1" />
     </link>
+    <link name="end_effector">
+        <xacro:boxTemplate x="${zetaJointRadius / 4}" y="${zetaJointRadius / 4}" z="${endEffectorZ}"
+            roll="0" pitch="0" yaw="0" ox="${zetaJointRadius * 3 / 4}" oy="0" oz="${zetaJointZ}" color="white" />
+        <xacro:defaultInertial mass="1" />
+    </link>
     <joint name="world_joint" type="fixed">
         <parent link="world" />
@@ -290,4 +296,8 @@
         <limit  effort="1000.00" lower="-2.36" upper="2.36" velocity="0.5" />
         <origin rpy="0 0 0" xyz="0 ${epsilonJointRadius1 + epsilonJointOffset1} ${epsilonJointZ1}" />
+    </joint>
+    <joint name="end_effector_joint" type="fixed">
+        <parent link="zeta_link" />
+        <child link="end_effector" />
     </joint>
     <!-- Gazebo plugin for ROS Control -->

Commit message: Changes to the simulation for towers of hannoi

File: urdf/andreas_arm_description.xacro (robot description, xacro)
@@ -103,11 +103,38 @@
     <link name="world" />
     <link name="base_link">
-        <xacro:cylinderTemplate length="${baseZ}" radius="${baseRadius}" roll="0" pitch="0" yaw="0" ox="0" oy="0" oz="${baseZ / 2}" color="white" />
+        <xacro:cylinderTemplate
+	    length="${baseZ}"
+	    radius="${baseRadius}"
+	    roll="0"
+	    pitch="0"
+	    yaw="0"
+	    ox="0"
+	    oy="0"
+	    oz="${baseZ / 2}"
+	    color="white" />
         <xacro:defaultInertial mass="1000" />
     </link>
     <link name="alpha_link">
         <!-- Shaft -->
-        <xacro:cylinderTemplate length="${alphaZ0}" radius="${alphaRadius0}" roll="0" pitch="0" yaw="0" ox="0" oy="0" oz="${alphaZ0 / 2}" color="white" />
-        <xacro:cylinderTemplate length="${alphaZ1}" radius="${alphaRadius1}" roll="0" pitch="0" yaw="0" ox="0" oy="0" oz="${alphaZ0 + alphaZ1 / 2}" color="white" />
+        <xacro:cylinderTemplate
+	    length="${alphaZ0}"
+	    radius="${alphaRadius0}"
+	    roll="0"
+	    pitch="0"
+	    yaw="0"
+	    ox="0"
+	    oy="0"
+	    oz="${alphaZ0 / 2}"
+	    color="white" />
+        <xacro:cylinderTemplate
+	    length="${alphaZ1}"
+	    radius="${alphaRadius1}"
+	    roll="0"
+	    pitch="0"
+	    yaw="0"
+	    ox="0"
+	    oy="0"
+	    oz="${alphaZ0 + alphaZ1 / 2}"
+	    color="white" />
         <!-- joint Hinge -->
         <xacro:boxTemplate x="${alphaJointX}" y="${alphaJointBlockY}" z="${alphaJointBlockZ}"

File: urdf/scorbot_description.xacro (robot description, xacro)
@@ -185,5 +185,5 @@
       lower="-0.6109"
       upper="2.2689"
-      effort="10"
+      effort="5"
       velocity="0.01587" />
   <!--0.4587-->
@@ -419,23 +419,21 @@
   </transmission>
     <link name="pad1_Link">
-        <xacro:defaultInertial mass="0.0001" />
-        <!--inertial>
-            <origin
-                xyz="-0.039374 5.5511E-17 -0.00025"
-                rpy="0 0 0" />
-            <mass value="0.007491" />
-            <inertia
-                ixx="1.655E-07"
-                ixy="-2.9699E-20"
-                ixz="-3.3353E-19"
-                iyy="3.5223E-06"
-                iyz="3.7058E-22"
-                izz="3.563E-06" />
-        </inertial-->
+        <inertial>
+            <origin xyz="0 0 0" rpy="0 0 0" />
+          <mass
+            value="0.0001" />
+          <inertia
+            ixx="0"
+            ixy="0"
+            ixz="0"
+            iyy="0"
+            iyz="0"
+            izz="0" />
+        </inertial>
         <visual>
             <geometry>
                 <box size="0.07 0.01 0.01" />
             </geometry>
-            <origin xyz="-0.035 0 0" rpy="0 0 0" />
+            <origin xyz="0 0 0" rpy="0 0 0" />
             <material name="">
                 <color rgba="0.1 0 0 1" />
@@ -446,58 +444,38 @@
                 <box size="0.07 0.01 0.01" />
             </geometry>
-            <origin xyz="-0.035 0 0" rpy="0 0 0" />
-            <material name="">
-                <color rgba="0.1 0 0 1" />
-            </material>
+            <origin xyz="0 0 0" rpy="0 0 0" />
+            <material name="">
+                <color rgba="0.1 0 0 1" />
+            </material>
+	    <friction>
+		<ode>
+		    <mu>100</mu>
+		    <mu2>100</mu2>
+		    <fdir1>0 0 0</fdir1>
+		    <slip1>0</slip1>
+		    <slip2>0</slip2>
+		</ode>
+	     </friction>
         </collision>
     </link>
-  <joint
-    name="pad1_joint"
-    type="revolute">
-    <origin
-      xyz="0 -0.0545 -0.0905"
-      rpy="1.5708 -0.74758 -1.5708" />
-    <parent
-      link="gripper_Link" />
-    <child
-      link="pad1_Link" />
-    <axis
-      xyz="0 0 1" />
-    <limit
-      lower="0"
-      upper="1.5709"
-      effort="100"
-      velocity="2" />
-  </joint>
-  <transmission name="pad1Transmission">
-    <type>transmission_interface/SimpleTransmission</type>
-    <joint name="pad1_joint" type="SimpleTransmission">
-      <hardwareInterface>EffortJointInterface</hardwareInterface>
-    </joint>
-    <actuator name="pad1_motor">
-      <machanicalReduction>1</machanicalReduction>
-      <hardwareInterface>EffortJointInterface</hardwareInterface>
-    </actuator>
-  </transmission>
     <link name="pad2_Link">
-        <xacro:defaultInertial mass="0.0001" />
-        <!--inertial>
-            <origin
-                xyz="-0.039374 -2.2204E-16 -0.00025"
-                rpy="0 0 0" />
-            <mass value="0.007491" />
-            <inertia
-                ixx="1.655E-07"
-                ixy="-2.9951E-20"
-                ixz="-3.496E-19"
-                iyy="3.5223E-06"
-                iyz="1.4029E-21"
-                izz="3.563E-06" />
-        </inertial-->
+        <!--xacro:defaultInertial mass="0.1" /-->
+        <inertial>
+            <origin xyz="0 0 0" rpy="0 0 0" />
+          <mass
+            value="0.0001" />
+          <inertia
+            ixx="0.00098187"
+            ixy="-2.7952E-20"
+            ixz="2.8189E-18"
+            iyy="0.00095638"
+            iyz="-2.4183E-18"
+            izz="0.00013429" />
+        </inertial>
         <visual>
             <geometry>
                 <box size="0.07 0.01 0.01" />
             </geometry>
-            <origin xyz="-0.035 0 0" rpy="0 0 0" />
+            <origin xyz="0 0 0" rpy="0 0 0" />
             <material name="">
                 <color rgba="0.1 0 0 1" />
@@ -508,38 +486,165 @@
                 <box size="0.07 0.01 0.01" />
             </geometry>
-            <origin xyz="-0.035 0 0" rpy="0 0 0" />
-            <material name="">
-                <color rgba="0.1 0 0 1" />
-            </material>
+            <origin xyz="0 0 0" rpy="0 0 0" />
+            <material name="">
+                <color rgba="0.1 0 0 1" />
+            </material>
+	    <friction>
+		<ode>
+		    <mu>100</mu>
+		    <mu2>100</mu2>
+		    <fdir1>0 0 0</fdir1>
+		    <slip1>0</slip1>
+		    <slip2>0</slip2>
+		</ode>
+	     </friction>
         </collision>
     </link>
-  <joint
-    name="pad2_joint"
-    type="revolute">
-    <origin
-      xyz="0 0.0545 -0.0905"
-      rpy="-1.5708 -0.74758 1.5708" />
-    <parent
-      link="gripper_Link" />
-    <child
-      link="pad2_Link" />
-    <axis
-      xyz="0 0 -1" />
-    <limit
-      lower="0"
-      upper="1.5709"
-      effort="100"
-      velocity="2" />
-  </joint>
-  <transmission name="pad2Transmission">
-    <type>transmission_interface/SimpleTransmission</type>
-    <joint name="pad2_joint" type="SimpleTransmission">
-      <hardwareInterface>EffortJointInterface</hardwareInterface>
-    </joint>
-    <actuator name="pad2_motor">
-      <machanicalReduction>1</machanicalReduction>
-      <hardwareInterface>EffortJointInterface</hardwareInterface>
-    </actuator>
-  </transmission>
+    <link name="pad1grip_Link">
+        <inertial>
+            <origin xyz="0 0 0" rpy="0 0 0" />
+          <mass
+            value="0.0000001" />
+          <inertia
+            ixx="0"
+            ixy="0"
+            ixz="0"
+            iyy="0"
+            iyz="0"
+            izz="0" />
+        </inertial>
+        <visual>
+            <geometry>
+                <box size="0.0001 0.01 0.01" />
+            </geometry>
+            <origin xyz="0.035 0 -0.01" rpy="0 0 0" />
+            <material name="">
+                <color rgba="0.1 0 0 1" />
+            </material>
+        </visual>
+        <collision>
+            <geometry>
+                <box size="0.0001 0.01 0.01" />
+            </geometry>
+            <origin xyz="0.035 0 -0.01" rpy="0 0 0" />
+            <material name="">
+                <color rgba="0.1 0 0 1" />
+            </material>
+	    <friction>
+		<ode>
+		    <mu>100</mu>
+		    <mu2>100</mu2>
+		    <fdir1>0 0 0</fdir1>
+		    <slip1>0</slip1>
+		    <slip2>0</slip2>
+		</ode>
+	     </friction>
+        </collision>
+    </link>
+    <link name="pad2grip_Link">
+        <inertial>
+            <origin xyz="0 0 0" rpy="0 0 0" />
+          <mass
+            value="0.0000001" />
+          <inertia
+            ixx="0"
+            ixy="0"
+            ixz="0"
+            iyy="0"
+            iyz="0"
+            izz="0" />
+        </inertial>
+        <visual>
+            <geometry>
+                <box size="0.0001 0.01 0.01" />
+            </geometry>
+            <origin xyz="0.035 0 -0.01" rpy="0 0 0" />
+            <material name="">
+                <color rgba="0.1 0 0 1" />
+            </material>
+        </visual>
+        <collision>
+            <geometry>
+                <box size="0.0001 0.01 0.01" />
+            </geometry>
+            <origin xyz="0.035 0 -0.01" rpy="0 0 0" />
+            <material name="">
+                <color rgba="0.1 0 0 1" />
+            </material>
+	    <friction>
+		<ode>
+		    <mu>100</mu>
+		    <mu2>100</mu2>
+		    <fdir1>0 0 0</fdir1>
+		    <slip1>0</slip1>
+		    <slip2>0</slip2>
+		</ode>
+	     </friction>
+        </collision>
+    </link>
+    <joint
+        name="pad1_joint"
+        type="prismatic">
+        <origin
+            xyz="0 0.005 -0.137"
+            rpy="0 1.5708 1.5708" />
+        <parent
+            link="gripper_Link" />
+        <child
+            link="pad1_Link" />
+        <axis
+            xyz="0 0 1" />
+        <limit
+            lower="0"
+            upper="0.0325"
+            effort="0.01"
+            velocity="1" />
+      </joint>
+      <joint
+          name="pad2_joint"
+          type="prismatic">
+        <origin
+            xyz="0 -0.005 -0.137"
+            rpy="0 1.5708 -1.5708" />
+        <parent
+            link="gripper_Link" />
+        <child
+            link="pad2_Link" />
+        <axis
+            xyz="0 0 1" />
+        <limit
+            lower="0"
+            upper="0.0325"
+            effort="0.01"
+            velocity="1" />
+      </joint>
+      <joint name="pad1grip_joint" type="fixed">
+	  <parent link="pad1_Link" />
+	  <child link="pad1grip_Link" />
+      </joint>
+      <joint name="pad2grip_joint" type="fixed">
+	  <parent link="pad2_Link" />
+	  <child link="pad2grip_Link" />
+      </joint>
+      <transmission name="pad1Transmission">
+          <type>transmission_interface/SimpleTransmission</type>
+          <joint name="pad1_joint" type="SimpleTransmission">
+              <hardwareInterface>EffortJointInterface</hardwareInterface>
+          </joint>
+          <actuator name="pad1_motor">
+              <machanicalReduction>1</machanicalReduction>
+              <hardwareInterface>EffortJointInterface</hardwareInterface>
+          </actuator>
+      </transmission>
+      <transmission name="pad2Transmission">
+          <type>transmission_interface/SimpleTransmission</type>
+          <joint name="pad2_joint" type="SimpleTransmission">
+              <hardwareInterface>EffortJointInterface</hardwareInterface>
+          </joint>
+          <actuator name="pad2_motor">
+              <machanicalReduction>1</machanicalReduction>
+              <hardwareInterface>EffortJointInterface</hardwareInterface>
+          </actuator>
+      </transmission>
     <!-- Gazebo plugin for ROS Control -->
     <gazebo>
@@ -554,5 +659,5 @@
                 <gripper_link>pad2_Link</gripper_link>
             </arm>
-            <forces_angle_tolerances>1</forces_angle_tolerances>
+            <forces_angle_tolerances>100</forces_angle_tolerances>
             <update_rate>4</update_rate>
             <grip_count_threshold>4</grip_count_threshold>
