Commit message: Integration of the ik with the drivers

File: urdf/scorbot_description.xacro (robot description, xacro)
@@ -116,5 +116,5 @@
       lower="-2.7054"
       upper="2.7054"
-      effort="5"
+      effort="5000"
       velocity="0.3488" />
     <dynamics
@@ -184,9 +184,9 @@
       link="elbow_Link" />
     <axis
-      xyz="1 0 0" />
-    <limit
-      lower="-2.2690"
-      upper="0.5236"
-      effort="4"
+      xyz="-1 0 0" />
+    <limit
+      lower="-0.6109"
+      upper="2.2689"
+      effort="400"
       velocity="0.4587" />
     <dynamics
@@ -256,9 +256,9 @@
       link="pitch_Link" />
     <axis
-      xyz="1 0 0" />
-    <limit
-      lower="-1.8327"
-      upper="2.2690"
-      effort="3"
+      xyz="-1 0 0" />
+    <limit
+      lower="-2.2689"
+      upper="2.2689"
+      effort="300"
       velocity="0.4587" />
     <dynamics
@@ -328,9 +328,9 @@
       link="roll_Link" />
     <axis
-      xyz="0 1 0" />
-    <limit
-      lower="-2.2690"
-      upper="2.2690"
-      effort="2"
+      xyz="0 -1 0" />
+    <limit
+      lower="-2.2689"
+      upper="2.2689"
+      effort="200"
       velocity="1.4478" />
     <dynamics
@@ -404,5 +404,5 @@
       lower="-9.9490"
       upper="9.9490"
-      effort="2"
+      effort="200"
       velocity="1.8491" />
     <dynamics
@@ -476,5 +476,5 @@
       lower="0"
       upper="1.5709"
-      effort="1"
+      effort="100"
       velocity="2" />
     <dynamics
@@ -548,5 +548,5 @@
       lower="0"
       upper="1.5709"
-      effort="1"
+      effort="100"
       velocity="2" />
     <dynamics

Commit message: Addition of a new gripper which works.

File: urdf/scorbot_description.xacro (robot description, xacro)
@@ -2,5 +2,5 @@
 <robot xmlns:xacro="http://www.ros.org/wiki/xacro" name="scorbot_model">
   <xacro:macro name="defaultInertial" params="mass">
-    <inertial>
+    <!--inertial>
       <mass value="${mass}" />
       <inertia
@@ -11,5 +11,5 @@
         iyz="0.0"
         izz="1.0" />
-    </inertial>
+    </inertial-->
   </xacro:macro>
   <link
@@ -393,6 +393,6 @@
     type="revolute">
     <origin
-      xyz="0 0 0"
-      rpy="0 1.3878E-17 0" />
+      xyz="0 0 0.01"
+      rpy="0 0 0" />
     <parent
       link="roll_Link" />
@@ -402,7 +402,7 @@
       xyz="0 0 1" />
     <limit
-      lower="-9.9490"
-      upper="9.9490"
-      effort="2"
+      lower="-1000"
+      upper="1000"
+      effort="1"
       velocity="1.8491" />
     <dynamics
@@ -420,6 +420,6 @@
     </actuator>
   </transmission>
-  <link
-    name="pad1_Link">
+  <!--link
+    name="lpad_Link">
     <inertial>
       <origin
@@ -438,5 +438,5 @@
     <visual>
       <origin
-        xyz="0 0 0"
+        xyz="0 0 0.0001"
         rpy="0 0 0" />
       <geometry>
@@ -452,5 +452,5 @@
     <collision>
       <origin
-        xyz="0 0 0"
+        xyz="0 0 0.0001"
         rpy="0 0 0" />
       <geometry>
@@ -459,16 +459,48 @@
       </geometry>
     </collision>
-    <xacro:defaultInertial mass="1" />
-  </link>
+  </link-->
+    <link name="lpad_Link">
+        <inertial>
+            <mass value="0.007491" />
+            <inertia
+                ixx="1.0"
+                ixy="0.0"
+                ixz="0.0"
+                iyy="1.0"
+                iyz="0.0"
+                izz="1.0" />
+        </inertial>
+        <visual>
+            <geometry>
+                <box size="0.06 0.01 0.01" />
+            </geometry>
+            <origin xyz="-0.03 0 0" rpy="0 0 0" />
+            <material name="">
+                <color rgba="0.1 0 0 1" />
+            </material>
+        </visual>
+        <collision>
+            <geometry>
+                <box size="0.05 0.01 0.01" />
+            </geometry>
+            <origin xyz="-0.03 0 0" rpy="0 0 0" />
+            <material name="">
+                <color rgba="0.1 0 0 1" />
+            </material>
+        </collision>
+    </link>
   <joint
-    name="pad1_joint"
+    name="lpad_joint"
     type="revolute">
     <origin
       xyz="0 -0.0545 -0.0905"
       rpy="1.5708 -0.74758 -1.5708" />
+    <!--origin
+      xyz="0 -0.0545 -0.0905"
+      rpy="1.5708 0 -1.5708" /-->
     <parent
       link="gripper_Link" />
     <child
-      link="pad1_Link" />
+      link="lpad_Link" />
     <axis
       xyz="0 0 1" />
@@ -476,5 +508,5 @@
       lower="0"
       upper="1.5709"
-      effort="1"
+      effort="0.5"
       velocity="2" />
     <dynamics
@@ -482,15 +514,15 @@
       friction="0.01" />
   </joint>
-  <transmission name="pad1Transmission">
+  <transmission name="lpadTransmission">
     <type>transmission_interface/SimpleTransmission</type>
-    <joint name="pad1_joint" type="SimpleTransmission">
+    <joint name="lpad_joint" type="SimpleTransmission">
       <hardwareInterface>EffortJointInterface</hardwareInterface>
     </joint>
-    <actuator name="pad1_motor">
+    <actuator name="lpad_motor">
       <machanicalReduction>1</machanicalReduction>
       <hardwareInterface>EffortJointInterface</hardwareInterface>
     </actuator>
   </transmission>
-  <link
+  <!--link
     name="pad2_Link">
     <inertial>
@@ -532,7 +564,37 @@
     </collision>
     <xacro:defaultInertial mass="1" />
-  </link>
+  </link-->
+    <link name="rpad_Link">
+        <inertial>
+            <mass value="0.007491" />
+            <inertia
+                ixx="1.0"
+                ixy="0.0"
+                ixz="0.0"
+                iyy="1.0"
+                iyz="0.0"
+                izz="1.0" />
+        </inertial>
+        <visual>
+            <geometry>
+                <box size="0.06 0.01 0.01" />
+            </geometry>
+            <origin xyz="-0.03 0 0" rpy="0 0 0" />
+            <material name="">
+                <color rgba="0.1 0 0 1" />
+            </material>
+        </visual>
+        <collision>
+            <geometry>
+                <box size="0.05 0.01 0.01" />
+            </geometry>
+            <origin xyz="-0.03 0 0" rpy="0 0 0" />
+            <material name="">
+                <color rgba="0.1 0 0 1" />
+            </material>
+        </collision>
+    </link>
   <joint
-    name="pad2_joint"
+    name="rpad_joint"
     type="revolute">
     <origin
@@ -542,5 +604,5 @@
       link="gripper_Link" />
     <child
-      link="pad2_Link" />
+      link="rpad_Link" />
     <axis
       xyz="0 0 -1" />
@@ -554,10 +616,10 @@
       friction="0.01" />
   </joint>
-  <transmission name="pad2Transmission">
+  <transmission name="rpadTransmission">
     <type>transmission_interface/SimpleTransmission</type>
-    <joint name="pad2_joint" type="SimpleTransmission">
+    <joint name="rpad_joint" type="SimpleTransmission">
       <hardwareInterface>EffortJointInterface</hardwareInterface>
     </joint>
-    <actuator name="pad2_motor">
+    <actuator name="rpad_motor">
       <machanicalReduction>1</machanicalReduction>
       <hardwareInterface>EffortJointInterface</hardwareInterface>

Commit message: ik changes

File: urdf/scorbot_description.xacro (robot description, xacro)
@@ -1,16 +1,4 @@
 <?xml version="1.0"?>
 <robot xmlns:xacro="http://www.ros.org/wiki/xacro" name="scorbot_model">
-  <xacro:macro name="defaultInertial" params="mass">
-    <!--inertial>
-      <mass value="${mass}" />
-      <inertia
-        ixx="1.0"
-        ixy="0.0"
-        ixz="0.0"
-        iyy="1.0"
-        iyz="0.0"
-        izz="1.0" />
-    </inertial-->
-  </xacro:macro>
   <link
       name="world" />
@@ -54,5 +42,4 @@
       </geometry>
     </collision>
-    <xacro:defaultInertial mass="1" />
   </link>
   <joint name="world_joint" type="fixed">
@@ -99,5 +86,4 @@
       </geometry>
     </collision>
-    <xacro:defaultInertial mass="1" />
   </link>
   <joint
@@ -116,5 +102,5 @@
       lower="-2.7054"
       upper="2.7054"
-      effort="500"
+      effort="5"
       velocity="0.3488" />
     <dynamics
@@ -171,5 +157,4 @@
       </geometry>
     </collision>
-    <xacro:defaultInertial mass="1" />
   </link>
   <joint
@@ -188,5 +173,5 @@
       lower="-0.6109"
       upper="2.2689"
-      effort="1600"
+      effort="16"
       velocity="0.4587" />
     <dynamics
@@ -243,5 +228,4 @@
       </geometry>
     </collision>
-    <xacro:defaultInertial mass="1" />
   </link>
   <joint
@@ -260,5 +244,5 @@
       lower="-2.2689"
       upper="2.2689"
-      effort="300"
+      effort="3"
       velocity="0.4587" />
     <dynamics
@@ -315,5 +299,4 @@
       </geometry>
     </collision>
-    <xacro:defaultInertial mass="1" />
   </link>
   <joint
@@ -387,5 +370,4 @@
       </geometry>
     </collision>
-    <xacro:defaultInertial mass="1" />
   </link>
   <joint
@@ -404,5 +386,5 @@
       lower="-1000"
       upper="1000"
-      effort="1"
+      effort="4"
       velocity="1.8491" />
     <dynamics
@@ -462,18 +444,21 @@
     <link name="lpad_Link">
         <inertial>
+            <origin
+                xyz="-0.039374 5.5511E-17 -0.00025"
+                rpy="0 0 0" />
             <mass value="0.007491" />
             <inertia
-                ixx="1.0"
-                ixy="0.0"
-                ixz="0.0"
-                iyy="1.0"
-                iyz="0.0"
-                izz="1.0" />
+                ixx="1.655E-07"
+                ixy="-2.9699E-20"
+                ixz="-3.3353E-19"
+                iyy="3.5223E-06"
+                iyz="3.7058E-22"
+                izz="3.563E-06" />
         </inertial>
         <visual>
             <geometry>
-                <box size="0.06 0.01 0.01" />
+                <box size="0.07 0.01 0.01" />
             </geometry>
-            <origin xyz="-0.03 0 0" rpy="0 0 0" />
+            <origin xyz="-0.035 0 0" rpy="0 0 0" />
             <material name="">
                 <color rgba="0.1 0 0 1" />
@@ -481,8 +466,8 @@
         </visual>
         <collision>
+            <origin xyz="-0.035 0 0" rpy="0 0 0" />
             <geometry>
-                <box size="0.05 0.01 0.01" />
+                <box size="0.07 0.01 0.01" />
             </geometry>
-            <origin xyz="-0.03 0 0" rpy="0 0 0" />
             <material name="">
                 <color rgba="0.1 0 0 1" />
@@ -508,5 +493,5 @@
       lower="0"
       upper="1.5709"
-      effort="0.5"
+      effort="4"
       velocity="2" />
     <dynamics
@@ -567,18 +552,21 @@
     <link name="rpad_Link">
         <inertial>
+            <origin
+                xyz="-0.039374 -2.2204E-16 -0.00025"
+                rpy="0 0 0" />
             <mass value="0.007491" />
             <inertia
-                ixx="1.0"
-                ixy="0.0"
-                ixz="0.0"
-                iyy="1.0"
-                iyz="0.0"
-                izz="1.0" />
+                ixx="1.655E-07"
+                ixy="-2.9951E-20"
+                ixz="-3.496E-19"
+                iyy="3.5223E-06"
+                iyz="1.4029E-21"
+                izz="3.563E-06" />
         </inertial>
         <visual>
             <geometry>
-                <box size="0.06 0.01 0.01" />
+                <box size="0.07 0.01 0.01" />
             </geometry>
-            <origin xyz="-0.03 0 0" rpy="0 0 0" />
+            <origin xyz="-0.035 0 0" rpy="0 0 0" />
             <material name="">
                 <color rgba="0.1 0 0 1" />
@@ -587,7 +575,7 @@
         <collision>
             <geometry>
-                <box size="0.05 0.01 0.01" />
+                <box size="0.07 0.01 0.01" />
             </geometry>
-            <origin xyz="-0.03 0 0" rpy="0 0 0" />
+            <origin xyz="-0.035 0 0" rpy="0 0 0" />
             <material name="">
                 <color rgba="0.1 0 0 1" />
@@ -610,5 +598,5 @@
       lower="0"
       upper="1.5709"
-      effort="1"
+      effort="4"
       velocity="2" />
     <dynamics

Commit message: Changes to the hand driver and launch files

File: urdf/scorbot_description.xacro (robot description, xacro)
@@ -173,5 +173,5 @@
       lower="-0.6109"
       upper="2.2689"
-      effort="16"
+      effort="100"
       velocity="0.4587" />
     <dynamics
@@ -244,5 +244,5 @@
       lower="-2.2689"
       upper="2.2689"
-      effort="3"
+      effort="25"
       velocity="0.4587" />
     <dynamics
@@ -403,5 +403,5 @@
   </transmission>
   <!--link
-    name="lpad_Link">
+    name="pad1_Link">
     <inertial>
       <origin
@@ -442,5 +442,5 @@
     </collision>
   </link-->
-    <link name="lpad_Link">
+    <link name="pad1_Link">
         <inertial>
             <origin
@@ -476,5 +476,5 @@
     </link>
   <joint
-    name="lpad_joint"
+    name="pad1_joint"
     type="revolute">
     <origin
@@ -487,5 +487,5 @@
       link="gripper_Link" />
     <child
-      link="lpad_Link" />
+      link="pad1_Link" />
     <axis
       xyz="0 0 1" />
@@ -493,5 +493,5 @@
       lower="0"
       upper="1.5709"
-      effort="4"
+      effort="1"
       velocity="2" />
     <dynamics
@@ -499,10 +499,10 @@
       friction="0.01" />
   </joint>
-  <transmission name="lpadTransmission">
+  <transmission name="pad1Transmission">
     <type>transmission_interface/SimpleTransmission</type>
-    <joint name="lpad_joint" type="SimpleTransmission">
+    <joint name="pad1_joint" type="SimpleTransmission">
       <hardwareInterface>EffortJointInterface</hardwareInterface>
     </joint>
-    <actuator name="lpad_motor">
+    <actuator name="pad1_motor">
       <machanicalReduction>1</machanicalReduction>
       <hardwareInterface>EffortJointInterface</hardwareInterface>
@@ -550,5 +550,5 @@
     <xacro:defaultInertial mass="1" />
   </link-->
-    <link name="rpad_Link">
+    <link name="pad2_Link">
         <inertial>
             <origin
@@ -584,5 +584,5 @@
     </link>
   <joint
-    name="rpad_joint"
+    name="pad2_joint"
     type="revolute">
     <origin
@@ -592,5 +592,5 @@
       link="gripper_Link" />
     <child
-      link="rpad_Link" />
+      link="pad2_Link" />
     <axis
       xyz="0 0 -1" />
@@ -598,5 +598,5 @@
       lower="0"
       upper="1.5709"
-      effort="4"
+      effort="1"
       velocity="2" />
     <dynamics
@@ -604,10 +604,10 @@
       friction="0.01" />
   </joint>
-  <transmission name="rpadTransmission">
+  <transmission name="pad2Transmission">
     <type>transmission_interface/SimpleTransmission</type>
-    <joint name="rpad_joint" type="SimpleTransmission">
+    <joint name="pad2_joint" type="SimpleTransmission">
       <hardwareInterface>EffortJointInterface</hardwareInterface>
     </joint>
-    <actuator name="rpad_motor">
+    <actuator name="pad2_motor">
       <machanicalReduction>1</machanicalReduction>
       <hardwareInterface>EffortJointInterface</hardwareInterface>
