Commit message: Towers of Hanoi now works.

File: urdf/scorbot_description.xacro (robot description, xacro)
@@ -16,5 +16,5 @@
         rpy="0 0 0" />
       <mass
-        value="0.001" />
+        value="13.939" />
       <inertia
         ixx="0.10125"
@@ -27,5 +27,5 @@
     <visual>
       <origin
-        xyz="0 0 0.010"
+        xyz="0 0 0.020"
         rpy="0 0 0" />
       <geometry>
@@ -42,5 +42,5 @@
     <collision>
       <origin
-        xyz="0 0 0.010"
+        xyz="0 0 0.020"
         rpy="0 0 0" />
       <geometry>
@@ -65,5 +65,5 @@
         rpy="0 0 0" /-->
       <mass
-        value="0.001" />
+        value="0.01" />
       <inertia
         ixx="0.069345"
@@ -102,5 +102,5 @@
     type="revolute">
     <origin
-      xyz="0 0 0.160"
+      xyz="0 0 0.165"
       rpy="0 0 0" />
     <parent
@@ -117,5 +117,5 @@
   <!--0.3488-->
     <dynamics
-      damping="0.01"
+      damping="0.0"
       friction="0.01" />
   </joint>
@@ -403,5 +403,4 @@
       effort="100"
       velocity="0.08491" />
-  <!--18491-->
     <dynamics
       damping="0.01"
@@ -433,5 +432,5 @@
         <visual>
             <geometry>
-                <box size="0.07 0.01 0.01" />
+                <box size="0.05 0.01 0.01" />
             </geometry>
             <origin xyz="0 0 0" rpy="0 0 0" />
@@ -442,5 +441,5 @@
         <collision>
             <geometry>
-                <box size="0.07 0.01 0.01" />
+                <box size="0.05 0.01 0.01" />
             </geometry>
             <origin xyz="0 0 0" rpy="0 0 0" />
@@ -460,5 +459,4 @@
     </link>
     <link name="pad2_Link">
-        <!--xacro:defaultInertial mass="0.1" /-->
         <inertial>
             <origin xyz="0 0 0" rpy="0 0 0" />
@@ -475,5 +473,5 @@
         <visual>
             <geometry>
-                <box size="0.07 0.01 0.01" />
+                <box size="0.05 0.01 0.01" />
             </geometry>
             <origin xyz="0 0 0" rpy="0 0 0" />
@@ -484,89 +482,7 @@
         <collision>
             <geometry>
-                <box size="0.07 0.01 0.01" />
+                <box size="0.05 0.01 0.01" />
             </geometry>
             <origin xyz="0 0 0" rpy="0 0 0" />
-            <material name="">
-                <color rgba="0.1 0 0 1" />
-            </material>
-	    <friction>
-		<ode>
-		    <mu>100</mu>
-		    <mu2>100</mu2>
-		    <fdir1>0 0 0</fdir1>
-		    <slip1>0</slip1>
-		    <slip2>0</slip2>
-		</ode>
-	     </friction>
-        </collision>
-    </link>
-    <link name="pad1grip_Link">
-        <inertial>
-            <origin xyz="0 0 0" rpy="0 0 0" />
-          <mass
-            value="0.0000001" />
-          <inertia
-            ixx="0"
-            ixy="0"
-            ixz="0"
-            iyy="0"
-            iyz="0"
-            izz="0" />
-        </inertial>
-        <visual>
-            <geometry>
-                <box size="0.0001 0.01 0.01" />
-            </geometry>
-            <origin xyz="0.035 0 -0.01" rpy="0 0 0" />
-            <material name="">
-                <color rgba="0.1 0 0 1" />
-            </material>
-        </visual>
-        <collision>
-            <geometry>
-                <box size="0.0001 0.01 0.01" />
-            </geometry>
-            <origin xyz="0.035 0 -0.01" rpy="0 0 0" />
-            <material name="">
-                <color rgba="0.1 0 0 1" />
-            </material>
-	    <friction>
-		<ode>
-		    <mu>100</mu>
-		    <mu2>100</mu2>
-		    <fdir1>0 0 0</fdir1>
-		    <slip1>0</slip1>
-		    <slip2>0</slip2>
-		</ode>
-	     </friction>
-        </collision>
-    </link>
-    <link name="pad2grip_Link">
-        <inertial>
-            <origin xyz="0 0 0" rpy="0 0 0" />
-          <mass
-            value="0.0000001" />
-          <inertia
-            ixx="0"
-            ixy="0"
-            ixz="0"
-            iyy="0"
-            iyz="0"
-            izz="0" />
-        </inertial>
-        <visual>
-            <geometry>
-                <box size="0.0001 0.01 0.01" />
-            </geometry>
-            <origin xyz="0.035 0 -0.01" rpy="0 0 0" />
-            <material name="">
-                <color rgba="0.1 0 0 1" />
-            </material>
-        </visual>
-        <collision>
-            <geometry>
-                <box size="0.0001 0.01 0.01" />
-            </geometry>
-            <origin xyz="0.035 0 -0.01" rpy="0 0 0" />
             <material name="">
                 <color rgba="0.1 0 0 1" />
@@ -587,5 +503,5 @@
         type="prismatic">
         <origin
-            xyz="0 0.005 -0.137"
+            xyz="0 0.005 -0.127"
             rpy="0 1.5708 1.5708" />
         <parent
@@ -598,5 +514,5 @@
             lower="0"
             upper="0.0325"
-            effort="0.01"
+            effort="0.001"
             velocity="1" />
       </joint>
@@ -605,5 +521,5 @@
           type="prismatic">
         <origin
-            xyz="0 -0.005 -0.137"
+            xyz="0 -0.005 -0.127"
             rpy="0 1.5708 -1.5708" />
         <parent
@@ -616,14 +532,6 @@
             lower="0"
             upper="0.0325"
-            effort="0.01"
+            effort="0.001"
             velocity="1" />
-      </joint>
-      <joint name="pad1grip_joint" type="fixed">
-	  <parent link="pad1_Link" />
-	  <child link="pad1grip_Link" />
-      </joint>
-      <joint name="pad2grip_joint" type="fixed">
-	  <parent link="pad2_Link" />
-	  <child link="pad2grip_Link" />
       </joint>
       <transmission name="pad1Transmission">
@@ -659,10 +567,10 @@
                 <gripper_link>pad2_Link</gripper_link>
             </arm>
-            <forces_angle_tolerances>100</forces_angle_tolerances>
+            <forces_angle_tolerance>100</forces_angle_tolerance>
             <update_rate>4</update_rate>
             <grip_count_threshold>4</grip_count_threshold>
             <max_grip_count>8</max_grip_count>
-            <release_tolerance>0.005</release_tolerance>
-            <disable_collisions_on_attach>true</disable_collisions_on_attach>
+            <release_tolerance>0.010</release_tolerance>
+            <disable_collisions_on_attach>false</disable_collisions_on_attach>
             <contact_topic>__default_topic__</contact_topic>
         </plugin>
